File: hardware/MCP73831.sch (KiCad schematic (older format))
At the start: 14 parts

Commit message: repair MCP73831,
Parts:
- removed C?: CP47uf,16V, Capacitor_SMD:CP_Elec_5x5.3, symbol taobao-cp:CP47uf,16V
- removed D? (x2): D_1N4148_T4, Diode_SMD:D_SOD-123, symbol taobao-d:D_1N4148_T4
- removed D?: LED_RED,0603, footprint-lib:LED_0603_1608Metric, symbol taobao-led:LED_RED,0603
- removed D?: LED_GREEN,0603, footprint-lib:LED_0603_1608Metric, symbol taobao-led:LED_GREEN,0603
- removed D?: LED_ORANGE,0603, footprint-lib:LED_0603_1608Metric, symbol taobao-led:LED_ORANGE,0603
- removed F?: Fuse_Small, symbol Device:Fuse_Small
- removed R? (x4): R122,0603, Resistor_SMD:R_0603_1608Metric_Pad1.05x0.95mm_HandSolder, symbol taobao-r:R122,0603
- removed R?: R103,0603, Resistor_SMD:R_0603_1608Metric_Pad1.05x0.95mm_HandSolder, symbol taobao-r:R103,0603
- removed U?: MCP73837_MSOP10, footprint-lib:MCP73837_MSOP10, symbol taobao-components:MCP73837_MSOP10
- removed U?: USB_Micro, footprint-lib:USB_Micro-B_Molex-105017-0001, symbol taobao-components:USB_Micro
- added C?: C106,0603, Capacitor_SMD:C_0603_1608Metric_Pad1.05x0.95mm_HandSolder, symbol taobao-c:C106,0603
- added D?: CHARGING, footprint-lib:LED_0603_1608Metric, symbol taobao-led:LED_ORANGE,0603
- added D?: D_1N4148_T4, Diode_SMD:D_SOD-123, symbol taobao-d:D_1N4148_T4
- added JP?: 5V_EN, Jumper:SolderJumper-2_P1.3mm_Open_RoundedPad1.0x1.5mm, symbol my_solder_jumper:SolderJumper_2_Open_round
- added JP?: SolderJumper_2_Open_round, Jumper:SolderJumper-2_P1.3mm_Open_RoundedPad1.0x1.5mm, symbol my_solder_jumper:SolderJumper_2_Open_round
- added R?: R102,0603, Resistor_SMD:R_0603_1608Metric_Pad1.05x0.95mm_HandSolder, symbol taobao-r:R102,0603
- added R?: R103,0603, Resistor_SMD:R_0603_1608Metric_Pad1.05x0.95mm_HandSolder, symbol taobao-r:R103,0603
- added U?: MCP73831, symbol taobao-components:MCP73831
Connections:
- net labels added: +5V, Vbat
- net labels removed: Vout
- wire segments 41 -> 21
