File: hardware/MCP73831.sch (KiCad schematic (older format))
At the start: 8 parts

Commit message: update,
Parts:
- JP2: renamed from JP?; value SolderJumper_2_Open_round -> OUT_EN
- U1: renamed from U?; footprint (none) -> footprint-lib:MCP73831_SOT23_5
- gave numbers to parts that had none: 6
Other:
- moved on the sheet: C1, D1, JP2, R2
Changed lines of the file:
@@
 $EndBitmap
 $Comp
-L taobao-components:MCP73831 U?
+L taobao-components:MCP73831 U1
 U 1 1 5CFFF5AE
 P 4450 2050
-F 0 "U?" H 4500 2500 50  0000 C CNN
+F 0 "U1" H 4500 2500 50  0000 C CNN
 F 1 "MCP73831" H 4500 2400 50  0000 C CNN
-F 2 "" H 4450 2050 50  0001 C CNN
+F 2 "footprint-lib:MCP73831_SOT23_5" H 4450 2050 50  0001 C CNN
 F 3 "" H 4450 2050 50  0001 C CNN
 	1    4450 2050
@@
 $EndComp
 $Comp
-L power:+5V #PWR?
+L power:+5V #PWR0101
 U 1 1 5CFFF8A1
 P 2700 1450
-F 0 "#PWR?" H 2700 1300 50  0001 C CNN
+F 0 "#PWR0101" H 2700 1300 50  0001 C CNN
 F 1 "+5V" H 2750 1650 50  0000 C CNN
 F 2 "" H 2700 1450 50  0001 C CNN
@@
 $EndComp
 $Comp
-L my_solder_jumper:SolderJumper_2_Open_round JP?
+L my_solder_jumper:SolderJumper_2_Open_round JP1
 U 1 1 5CFFFF75
 P 2700 1700
-F 0 "JP?" V 2650 1800 50  0000 L CNN
+F 0 "JP1" V 2650 1800 50  0000 L CNN
 F 1 "5V_EN" V 2700 1800 50  0000 L CNN
 F 2 "Jumper:SolderJumper-2_P1.3mm_Open_RoundedPad1.0x1.5mm" H 2700 1700 50  0001 C CNN
@@
 $EndComp
 $Comp
-L taobao-led:LED_ORANGE,0603 D?
+L taobao-led:LED_ORANGE,0603 D2
 U 1 1 5D0007CF
 P 3000 2150
-F 0 "D?" H 3000 2300 50  0000 C CNN
+F 0 "D2" H 3000 2300 50  0000 C CNN
 F 1 "CHARGING" H 3000 2400 50  0000 C CNN
 F 2 "footprint-lib:LED_0603_1608Metric" V 3000 2150 50  0001 C CNN
@@
 $EndComp
 $Comp
-L taobao-r:R102,0603 R?
+L taobao-r:R102,0603 R1
 U 1 1 5D0011EB
 P 3550 2150
-F 0 "R?" V 3700 2150 50  0000 C CNN
+F 0 "R1" V 3700 2150 50  0000 C CNN
 F 1 "R102,0603" V 3800 2150 50  0000 C CNN
 F 2 "Resistor_SMD:R_0603_1608Metric_Pad1.05x0.95mm_HandSolder" H 3550 2150 50  0001 C CNN
@@
 	2700 1950 2700 2150
 $Comp
-L my_solder_jumper:SolderJumper_2_Open_round JP?
+L my_solder_jumper:SolderJumper_2_Open_round JP2
 U 1 1 5D001D05
-P 5400 1900
-F 0 "JP?" H 5400 2150 50  0000 C CNN
-F 1 "SolderJumper_2_Open_round" H 5400 2050 50  0000 C CNN
-F 2 "Jumper:SolderJumper-2_P1.3mm_Open_RoundedPad1.0x1.5mm" H 5400 1900 50  0001 C CNN
-F 3 "~" H 5400 1900 50  0001 C CNN
-	1    5400 1900
-	1    0    0    -1
-$EndComp
-$Comp
-L my_power:Vbat #PWR?
+P 5200 1700
+F 0 "JP2" H 5200 1950 50  0000 C CNN
+F 1 "OUT_EN" H 5200 1850 50  0000 C CNN
+F 2 "Jumper:SolderJumper-2_P1.3mm_Open_RoundedPad1.0x1.5mm" H 5200 1700 50  0001 C CNN
+F 3 "~" H 5200 1700 50  0001 C CNN
+	1    5200 1700
+	0    -1   -1   0
+$EndComp
+$Comp
+L my_power:Vbat #PWR0102
 U 1 1 5D002381
-P 6050 1650
-F 0 "#PWR?" H 6050 1500 50  0001 C CNN
-F 1 "Vbat" H 6100 1800 50  0000 C CNN
-F 2 "" H 6050 1650 50  0001 C CNN
-F 3 "" H 6050 1650 50  0001 C CNN
-	1    6050 1650
-	1    0    0    -1
-$EndComp
-Wire Wire Line
-	6050 1650 6050 1900
-Wire Wire Line
-	6050 1900 5850 1900
-Wire Wire Line
-	4900 1900 5250 1900
-$Comp
-L taobao-r:R103,0603 R?
+P 5400 1200
+F 0 "#PWR0102" H 5400 1050 50  0001 C CNN
+F 1 "Vbat" H 5450 1350 50  0000 C CNN
+F 2 "" H 5400 1200 50  0001 C CNN
+F 3 "" H 5400 1200 50  0001 C CNN
+	1    5400 1200
+	1    0    0    -1
+$EndComp
+Wire Wire Line
+	5400 1200 5400 1450
+Wire Wire Line
+	5400 1450 5200 1450
+Wire Wire Line
+	4900 1900 5200 1900
+$Comp
+L taobao-r:R103,0603 R2
 U 1 1 5D002BCB
-P 5350 2050
-F 0 "R?" V 5100 2050 50  0000 C CNN
-F 1 "R103,0603" V 5200 2050 50  0000 C CNN
-F 2 "Resistor_SMD:R_0603_1608Metric_Pad1.05x0.95mm_HandSolder" H 5350 2050 50  0001 C CNN
-F 3 "~" H 5350 2050 50  0001 C CNN
-	1    5350 2050
-	0    1    1    0
-$EndComp
-$Comp
-L taobao-c:C106,0603 C?
+P 5250 2200
+F 0 "R2" H 5150 2150 50  0000 R CNN
+F 1 "R103,0603" H 5150 2200 50  0000 R CNN
+F 2 "Resistor_SMD:R_0603_1608Metric_Pad1.05x0.95mm_HandSolder" H 5250 2200 50  0001 C CNN
+F 3 "~" H 5250 2200 50  0001 C CNN
+	1    5250 2200
+	-1   0    0    1
+$EndComp
+$Comp
+L taobao-c:C106,0603 C1
 U 1 1 5D003198
-P 5850 2300
-F 0 "C?" H 5950 2350 50  0000 L CNN
-F 1 "C106,0603" H 5950 2300 50  0000 L CNN
-F 2 "Capacitor_SMD:C_0603_1608Metric_Pad1.05x0.95mm_HandSolder" H 5850 2300 50  0001 C CNN
-F 3 "~" H 5850 2300 50  0001 C CNN
-	1    5850 2300
+P 5450 1800
+F 0 "C1" H 5550 1850 50  0000 L CNN
+F 1 "C106,0603" H 5550 1800 50  0000 L CNN
+F 2 "Capacitor_SMD:C_0603_1608Metric_Pad1.05x0.95mm_HandSolder" H 5450 1800 50  0001 C CNN
+F 3 "~" H 5450 1800 50  0001 C CNN
+	1    5450 1800
 	1    0    0    -1
 $EndComp
 Wire Wire Line
 	4900 2050 5250 2050
-Wire Wire Line
-	4900 2200 5600 2200
-Wire Wire Line
-	5600 2200 5600 2050
-Wire Wire Line
-	5600 2050 5450 2050
-$Comp
-L power:GND #PWR?
+$Comp
+L power:GND #PWR0103
 U 1 1 5D0039E3
-P 5600 2500
-F 0 "#PWR?" H 5600 2250 50  0001 C CNN
-F 1 "GND" H 5650 2300 50  0000 C CNN
-F 2 "" H 5600 2500 50  0001 C CNN
-F 3 "" H 5600 2500 50  0001 C CNN
-	1    5600 2500
-	1    0    0    -1
-$EndComp
-Wire Wire Line
-	5600 2500 5600 2200
-Connection ~ 5600 2200
-Wire Wire Line
-	5850 2200 5850 1900
-Connection ~ 5850 1900
-Wire Wire Line
-	5850 1900 5550 1900
-$Comp
-L power:GND #PWR?
+P 5250 2750
+F 0 "#PWR0103" H 5250 2500 50  0001 C CNN
+F 1 "GND" H 5300 2550 50  0000 C CNN
+F 2 "" H 5250 2750 50  0001 C CNN
+F 3 "" H 5250 2750 50  0001 C CNN
+	1    5250 2750
+	1    0    0    -1
+$EndComp
+$Comp
+L power:GND #PWR0104
 U 1 1 5D003EE4
-P 5850 2500
-F 0 "#PWR?" H 5850 2250 50  0001 C CNN
-F 1 "GND" H 5900 2300 50  0000 C CNN
-F 2 "" H 5850 2500 50  0001 C CNN
-F 3 "" H 5850 2500 50  0001 C CNN
-	1    5850 2500
-	1    0    0    -1
-$EndComp
-Wire Wire Line
-	5850 2400 5850 2500
-$Comp
-L taobao-d:D_1N4148_T4 D?
+P 5450 2000
+F 0 "#PWR0104" H 5450 1750 50  0001 C CNN
+F 1 "GND" H 5550 2000 50  0000 L CNN
+F 2 "" H 5450 2000 50  0001 C CNN
+F 3 "" H 5450 2000 50  0001 C CNN
+	1    5450 2000
+	1    0    0    -1
+$EndComp
+Wire Wire Line
+	5450 1900 5450 2000
+$Comp
+L taobao-d:D_1N4148_T4 D1
 U 1 1 5D004835
-P 6300 1900
-F 0 "D?" H 6300 1650 50  0000 C CNN
-F 1 "D_1N4148_T4" H 6300 1750 50  0000 C CNN
-F 2 "Diode_SMD:D_SOD-123" V 6300 1900 50  0001 C CNN
-F 3 "~" V 6300 1900 50  0001 C CNN
-	1    6300 1900
+P 5650 1450
+F 0 "D1" H 5650 1200 50  0000 C CNN
+F 1 "D_1N4148_T4" H 5650 1300 50  0000 C CNN
+F 2 "Diode_SMD:D_SOD-123" V 5650 1450 50  0001 C CNN
+F 3 "~" V 5650 1450 50  0001 C CNN
+	1    5650 1450
 	-1   0    0    1
 $EndComp
@@
 	2700 1450 2700 1550
 Wire Wire Line
-	6200 1900 6050 1900
-Connection ~ 6050 1900
-$Comp
-L power:+5V #PWR?
+	5550 1450 5450 1450
+Connection ~ 5400 1450
+$Comp
+L power:+5V #PWR0105
 U 1 1 5D007E6E
-P 6550 1700
-F 0 "#PWR?" H 6550 1550 50  0001 C CNN
-F 1 "+5V" H 6600 1900 50  0000 C CNN
-F 2 "" H 6550 1700 50  0001 C CNN
-F 3 "" H 6550 1700 50  0001 C CNN
-	1    6550 1700
-	1    0    0    -1
-$EndComp
-Wire Wire Line
-	6400 1900 6550 1900
-Wire Wire Line
-	6550 1900 6550 1700
+P 5900 1250
+F 0 "#PWR0105" H 5900 1100 50  0001 C CNN
+F 1 "+5V" H 5950 1450 50  0000 C CNN
+F 2 "" H 5900 1250 50  0001 C CNN
+F 3 "" H 5900 1250 50  0001 C CNN
+	1    5900 1250
+	1    0    0    -1
+$EndComp
+Wire Wire Line
+	5750 1450 5900 1450
+Wire Wire Line
+	5900 1450 5900 1250
 $Bitmap
 Pos -700 2250
@@
 EndData
 $EndBitmap
+Wire Wire Line
+	5200 1450 5200 1550
+Wire Wire Line
+	5200 1850 5200 1900
+Wire Wire Line
+	5250 2300 5250 2350
+Wire Wire Line
+	4900 2200 5000 2200
+Wire Wire Line
+	5000 2200 5000 2350
+Wire Wire Line
+	5000 2350 5250 2350
+Connection ~ 5250 2350
+Wire Wire Line
+	5250 2350 5250 2750
+Wire Wire Line
+	5250 2050 5250 2100
+Connection ~ 5450 1450
+Wire Wire Line
+	5450 1450 5400 1450
+Wire Wire Line
+	5450 1450 5450 1700
 $EndSCHEMATC

Commit message: update,
Parts:
- added J1: PWR_SRC, Connector_PinHeader_2.54mm:PinHeader_1x02_P2.54mm_Vertical, symbol Connector:Conn_01x02_Female
- added J2: 5V_OUT, Connector_PinHeader_2.54mm:PinHeader_1x02_P2.54mm_Vertical, symbol Connector:Conn_01x02_Female
- added J3: BAT, Connector_PinHeader_2.54mm:PinHeader_1x02_P2.54mm_Vertical, symbol Connector:Conn_01x02_Female
Connections:
- net +5V: now also J2.2 (Pin_2); no longer JP1.1 (A)
- net GND: now also J1.1 (Pin_1), J2.1 (Pin_1), J3.1 (Pin_1)
- net Vbat: now also J3.2 (Pin_2)
- new net VCC: J1.2 (Pin_2), JP1.1 (A)
Changed lines of the file:
@@
-$EndComp
-$Comp
-L power:+5V #PWR0101
-U 1 1 5CFFF8A1
-P 2700 1450
-F 0 "#PWR0101" H 2700 1300 50  0001 C CNN
-F 1 "+5V" H 2750 1650 50  0000 C CNN
-F 2 "" H 2700 1450 50  0001 C CNN
-F 3 "" H 2700 1450 50  0001 C CNN
-	1    2700 1450
-	1    0    0    -1
 $EndComp
 $Comp
@@
 Wire Wire Line
 	5450 1450 5450 1700
+$Comp
+L Connector:Conn_01x02_Female J1
+U 1 1 5D0903C7
+P 6500 1300
+F 0 "J1" H 6528 1276 50  0000 L CNN
+F 1 "PWR_SRC" H 6528 1185 50  0000 L CNN
+F 2 "Connector_PinHeader_2.54mm:PinHeader_1x02_P2.54mm_Vertical" H 6500 1300 50  0001 C CNN
+F 3 "~" H 6500 1300 50  0001 C CNN
+	1    6500 1300
+	1    0    0    -1
+$EndComp
+Wire Wire Line
+	6150 1550 6150 1400
+Wire Wire Line
+	6150 1400 6300 1400
+$Comp
+L power:GND #PWR0101
+U 1 1 5D0917CE
+P 6150 1200
+F 0 "#PWR0101" H 6150 950 50  0001 C CNN
+F 1 "GND" H 6155 1027 50  0000 C CNN
+F 2 "" H 6150 1200 50  0001 C CNN
+F 3 "" H 6150 1200 50  0001 C CNN
+	1    6150 1200
+	-1   0    0    1
+$EndComp
+Wire Wire Line
+	6150 1200 6150 1300
+Wire Wire Line
+	6150 1300 6300 1300
+$Comp
+L Connector:Conn_01x02_Female J2
+U 1 1 5D0924C9
+P 6500 2050
+F 0 "J2" H 6528 2026 50  0000 L CNN
+F 1 "5V_OUT" H 6528 1935 50  0000 L CNN
+F 2 "Connector_PinHeader_2.54mm:PinHeader_1x02_P2.54mm_Vertical" H 6500 2050 50  0001 C CNN
+F 3 "~" H 6500 2050 50  0001 C CNN
+	1    6500 2050
+	1    0    0    -1
+$EndComp
+$Comp
+L power:+5V #PWR0106
+U 1 1 5D0924D3
+P 6150 2300
+F 0 "#PWR0106" H 6150 2150 50  0001 C CNN
+F 1 "+5V" H 6200 2500 50  0000 C CNN
+F 2 "" H 6150 2300 50  0001 C CNN
+F 3 "" H 6150 2300 50  0001 C CNN
+	1    6150 2300
+	-1   0    0    1
+$EndComp
+Wire Wire Line
+	6150 2300 6150 2150
+Wire Wire Line
+	6150 2150 6300 2150
+$Comp
+L power:GND #PWR0107
+U 1 1 5D0924DF
+P 6150 1950
+F 0 "#PWR0107" H 6150 1700 50  0001 C CNN
+F 1 "GND" H 6155 1777 50  0000 C CNN
+F 2 "" H 6150 1950 50  0001 C CNN
+F 3 "" H 6150 1950 50  0001 C CNN
+	1    6150 1950
+	-1   0    0    1
+$EndComp
+Wire Wire Line
+	6150 1950 6150 2050
+Wire Wire Line
+	6150 2050 6300 2050
+$Comp
+L power:VCC #PWR0108
+U 1 1 5D095653
+P 2700 1450
+F 0 "#PWR0108" H 2700 1300 50  0001 C CNN
+F 1 "VCC" H 2717 1623 50  0000 C CNN
+F 2 "" H 2700 1450 50  0001 C CNN
+F 3 "" H 2700 1450 50  0001 C CNN
+	1    2700 1450
+	1    0    0    -1
+$EndComp
+$Comp
+L power:VCC #PWR0109
+U 1 1 5D0973AB
+P 6150 1550
+F 0 "#PWR0109" H 6150 1400 50  0001 C CNN
+F 1 "VCC" H 6168 1723 50  0000 C CNN
+F 2 "" H 6150 1550 50  0001 C CNN
+F 3 "" H 6150 1550 50  0001 C CNN
+	1    6150 1550
+	-1   0    0    1
+$EndComp
+$Comp
+L Connector:Conn_01x02_Female J3
+U 1 1 5D097E87
+P 6500 2800
+F 0 "J3" H 6528 2776 50  0000 L CNN
+F 1 "BAT" H 6528 2685 50  0000 L CNN
+F 2 "Connector_PinHeader_2.54mm:PinHeader_1x02_P2.54mm_Vertical" H 6500 2800 50  0001 C CNN
+F 3 "~" H 6500 2800 50  0001 C CNN
+	1    6500 2800
+	1    0    0    -1
+$EndComp
+Wire Wire Line
+	6150 3050 6150 2900
+Wire Wire Line
+	6150 2900 6300 2900
+$Comp
+L power:GND #PWR0110
+U 1 1 5D097E9D
+P 6150 2700
+F 0 "#PWR0110" H 6150 2450 50  0001 C CNN
+F 1 "GND" H 6155 2527 50  0000 C CNN
+F 2 "" H 6150 2700 50  0001 C CNN
+F 3 "" H 6150 2700 50  0001 C CNN
+	1    6150 2700
+	-1   0    0    1
+$EndComp
+Wire Wire Line
+	6150 2700 6150 2800
+Wire Wire Line
+	6150 2800 6300 2800
+$Comp
+L my_power:Vbat #PWR0111
+U 1 1 5D099450
+P 6150 3050
+F 0 "#PWR0111" H 6150 2900 50  0001 C CNN
+F 1 "Vbat" H 6155 3173 50  0000 C CNN
+F 2 "" H 6150 3050 50  0001 C CNN
+F 3 "" H 6150 3050 50  0001 C CNN
+	1    6150 3050
+	-1   0    0    1
+$EndComp
 $EndSCHEMATC

Commit message: update,
Parts:
- added C?: C106,0603, Capacitor_SMD:C_0603_1608Metric_Pad1.05x0.95mm_HandSolder, symbol taobao-c:C106,0603
- renumbered C1 to C?, D2 to D?, D1 to D?, J1 to J?, J2 to J?, J3 to J?, JP1 to JP?, JP2 to JP?, R1 to R?, R2 to R?, U1 to U?
Connections:
- net +5V: now also C?.1
- net GND: now also C?.2
- net Vbat: now also C?.1; no longer C?.1
- net VCC renamed VBUS
Other:
- moved on the sheet: C?, D?, JP?, R?, U?

Commit message: update,
Parts:
- gave numbers to parts that had none: 12
Changed lines of the file:
@@
 $EndBitmap
 $Comp
-L taobao-components:MCP73831 U?
+L taobao-components:MCP73831 U1
 U 1 1 5CFFF5AE
 P 2800 2150
-F 0 "U?" H 2850 2600 50  0000 C CNN
+F 0 "U1" H 2850 2600 50  0000 C CNN
 F 1 "MCP73831" H 2850 2500 50  0000 C CNN
 F 2 "footprint-lib:MCP73831_SOT23_5" H 2800 2150 50  0001 C CNN
@@
 $EndComp
 $Comp
-L my_solder_jumper:SolderJumper_2_Open_round JP?
+L my_solder_jumper:SolderJumper_2_Open_round JP1
 U 1 1 5CFFFF75
 P 1050 1800
-F 0 "JP?" V 1000 1900 50  0000 L CNN
+F 0 "JP1" V 1000 1900 50  0000 L CNN
 F 1 "5V_EN" V 1050 1900 50  0000 L CNN
 F 2 "Jumper:SolderJumper-2_P1.3mm_Open_RoundedPad1.0x1.5mm" H 1050 1800 50  0001 C CNN
@@
 $EndComp
 $Comp
-L taobao-led:LED_ORANGE,0603 D?
+L taobao-led:LED_ORANGE,0603 D2
 U 1 1 5D0007CF
 P 1350 2250
-F 0 "D?" H 1350 2400 50  0000 C CNN
+F 0 "D2" H 1350 2400 50  0000 C CNN
 F 1 "CHARGING" H 1350 2500 50  0000 C CNN
 F 2 "footprint-lib:LED_0603_1608Metric" V 1350 2250 50  0001 C CNN
@@
 $EndComp
 $Comp
-L taobao-r:R102,0603 R?
+L taobao-r:R102,0603 R1
 U 1 1 5D0011EB
 P 1900 2250
-F 0 "R?" V 2050 2250 50  0000 C CNN
+F 0 "R1" V 2050 2250 50  0000 C CNN
 F 1 "R102,0603" V 2150 2250 50  0000 C CNN
 F 2 "Resistor_SMD:R_0603_1608Metric_Pad1.05x0.95mm_HandSolder" H 1900 2250 50  0001 C CNN
@@
 	1050 2050 1050 2250
 $Comp
-L my_solder_jumper:SolderJumper_2_Open_round JP?
+L my_solder_jumper:SolderJumper_2_Open_round JP2
 U 1 1 5D001D05
 P 3700 2000
-F 0 "JP?" H 3700 2250 50  0000 C CNN
+F 0 "JP2" H 3700 2250 50  0000 C CNN
 F 1 "OUT_EN" H 3700 2150 50  0000 C CNN
 F 2 "Jumper:SolderJumper-2_P1.3mm_Open_RoundedPad1.0x1.5mm" H 3700 2000 50  0001 C CNN
@@
 $EndComp
 $Comp
-L my_power:Vbat #PWR?
+L my_power:Vbat #PWR0101
 U 1 1 5D002381
 P 4300 1750
-F 0 "#PWR?" H 4300 1600 50  0001 C CNN
+F 0 "#PWR0101" H 4300 1600 50  0001 C CNN
 F 1 "Vbat" H 4350 1900 50  0000 C CNN
 F 2 "" H 4300 1750 50  0001 C CNN
@@
 	3250 2000 3550 2000
 $Comp
-L taobao-r:R103,0603 R?
+L taobao-r:R103,0603 R2
 U 1 1 5D002BCB
 P 3600 2300
-F 0 "R?" H 3500 2250 50  0000 R CNN
+F 0 "R2" H 3500 2250 50  0000 R CNN
 F 1 "R103,0603" H 3500 2300 50  0000 R CNN
 F 2 "Resistor_SMD:R_0603_1608Metric_Pad1.05x0.95mm_HandSolder" H 3600 2300 50  0001 C CNN
@@
 	3250 2150 3600 2150
 $Comp
-L power:GND #PWR?
+L power:GND #PWR0102
 U 1 1 5D0039E3
 P 3600 2850
-F 0 "#PWR?" H 3600 2600 50  0001 C CNN
+F 0 "#PWR0102" H 3600 2600 50  0001 C CNN
 F 1 "GND" H 3650 2650 50  0000 C CNN
 F 2 "" H 3600 2850 50  0001 C CNN
@@
 	1050 1550 1050 1650
 $Comp
-L power:+5V #PWR?
+L power:+5V #PWR0103
 U 1 1 5D007E6E
 P 4850 1800
-F 0 "#PWR?" H 4850 1650 50  0001 C CNN
+F 0 "#PWR0103" H 4850 1650 50  0001 C CNN
 F 1 "+5V" H 4900 2000 50  0000 C CNN
 F 2 "" H 4850 1800 50  0001 C CNN
@@
 	3600 2150 3600 2200
 $Comp
-L Connector:Conn_01x02_Female J?
+L Connector:Conn_01x02_Female J3
 U 1 1 5D097E87
 P 6500 2800
-F 0 "J?" H 6528 2776 50  0000 L CNN
+F 0 "J3" H 6528 2776 50  0000 L CNN
 F 1 "BAT" H 6528 2685 50  0000 L CNN
 F 2 "Connector_PinHeader_2.54mm:PinHeader_1x02_P2.54mm_Vertical" H 6500 2800 50  0001 C CNN
@@
 	6150 2900 6300 2900
 $Comp
-L power:GND #PWR?
+L power:GND #PWR0104
 U 1 1 5D097E9D
 P 6150 2700
-F 0 "#PWR?" H 6150 2450 50  0001 C CNN
+F 0 "#PWR0104" H 6150 2450 50  0001 C CNN
 F 1 "GND" H 6155 2527 50  0000 C CNN
 F 2 "" H 6150 2700 50  0001 C CNN
@@
 	6150 2800 6300 2800
 $Comp
-L my_power:Vbat #PWR?
+L my_power:Vbat #PWR0105
 U 1 1 5D099450
 P 6150 3050
-F 0 "#PWR?" H 6150 2900 50  0001 C CNN
+F 0 "#PWR0105" H 6150 2900 50  0001 C CNN
 F 1 "Vbat" H 6155 3173 50  0000 C CNN
 F 2 "" H 6150 3050 50  0001 C CNN
@@
 	6150 1950 6150 2050
 $Comp
-L power:GND #PWR?
+L power:GND #PWR0106
 U 1 1 5D0924DF
 P 6150 1950
-F 0 "#PWR?" H 6150 1700 50  0001 C CNN
+F 0 "#PWR0106" H 6150 1700 50  0001 C CNN
 F 1 "GND" H 6155 1777 50  0000 C CNN
 F 2 "" H 6150 1950 50  0001 C CNN
@@
 	6150 2300 6150 2150
 $Comp
-L power:+5V #PWR?
+L power:+5V #PWR0107
 U 1 1 5D0924D3
 P 6150 2300
-F 0 "#PWR?" H 6150 2150 50  0001 C CNN
+F 0 "#PWR0107" H 6150 2150 50  0001 C CNN
 F 1 "+5V" H 6200 2500 50  0000 C CNN
 F 2 "" H 6150 2300 50  0001 C CNN
@@
 $EndComp
 $Comp
-L Connector:Conn_01x02_Female J?
+L Connector:Conn_01x02_Female J2
 U 1 1 5D0924C9
 P 6500 2050
-F 0 "J?" H 6528 2026 50  0000 L CNN
+F 0 "J2" H 6528 2026 50  0000 L CNN
 F 1 "5V_OUT" H 6528 1935 50  0000 L CNN
 F 2 "Connector_PinHeader_2.54mm:PinHeader_1x02_P2.54mm_Vertical" H 6500 2050 50  0001 C CNN
@@
 	6150 1200 6150 1300
 $Comp
-L power:GND #PWR?
+L power:GND #PWR0108
 U 1 1 5D0917CE
 P 6150 1200
-F 0 "#PWR?" H 6150 950 50  0001 C CNN
+F 0 "#PWR0108" H 6150 950 50  0001 C CNN
 F 1 "GND" H 6155 1027 50  0000 C CNN
 F 2 "" H 6150 1200 50  0001 C CNN
@@
 	6150 1550 6150 1400
 $Comp
-L Connector:Conn_01x02_Female J?
+L Connector:Conn_01x02_Female J1
 U 1 1 5D0903C7
 P 6500 1300
-F 0 "J?" H 6528 1276 50  0000 L CNN
+F 0 "J1" H 6528 1276 50  0000 L CNN
 F 1 "PWR_SRC" H 6528 1185 50  0000 L CNN
 F 2 "Connector_PinHeader_2.54mm:PinHeader_1x02_P2.54mm_Vertical" H 6500 1300 50  0001 C CNN
@@
 $EndComp
 $Comp
-L power:VBUS #PWR?
+L power:VBUS #PWR0109
 U 1 1 5D204CBD
 P 1050 1550
-F 0 "#PWR?" H 1050 1400 50  0001 C CNN
+F 0 "#PWR0109" H 1050 1400 50  0001 C CNN
 F 1 "VBUS" H 1065 1723 50  0000 C CNN
 F 2 "" H 1050 1550 50  0001 C CNN
@@
 $EndComp
 $Comp
-L power:VBUS #PWR?
+L power:VBUS #PWR0110
 U 1 1 5D205CEA
 P 6150 1550
-F 0 "#PWR?" H 6150 1400 50  0001 C CNN
+F 0 "#PWR0110" H 6150 1400 50  0001 C CNN
 F 1 "VBUS" H 6165 1723 50  0000 C CNN
 F 2 "" H 6150 1550 50  0001 C CNN
@@
 $EndComp
 $Comp
-L my_power:Vbat #PWR?
+L my_power:Vbat #PWR0111
 U 1 1 5D218F01
 P 5100 1450
-F 0 "#PWR?" H 5100 1300 50  0001 C CNN
+F 0 "#PWR0111" H 5100 1300 50  0001 C CNN
 F 1 "Vbat" H 5150 1600 50  0000 C CNN
 F 2 "" H 5100 1450 50  0001 C CNN
@@
 	3850 2000 4300 2000
 $Comp
-L taobao-d:D_1N4148_T4 D?
+L taobao-d:D_1N4148_T4 D1
 U 1 1 5D004835
 P 5100 1800
-F 0 "D?" H 5100 1550 50  0000 C CNN
+F 0 "D1" H 5100 1550 50  0000 C CNN
 F 1 "D_1N4148_T4" H 5100 1650 50  0000 C CNN
 F 2 "Diode_SMD:D_SOD-123" V 5100 1800 50  0001 C CNN
@@
 	5100 2450 5100 2550
 $Comp
-L power:GND #PWR?
+L power:GND #PWR0112
 U 1 1 5D003EE4
 P 5100 2550
-F 0 "#PWR?" H 5100 2300 50  0001 C CNN
+F 0 "#PWR0112" H 5100 2300 50  0001 C CNN
 F 1 "GND" H 5200 2550 50  0000 L CNN
 F 2 "" H 5100 2550 50  0001 C CNN
@@
 $EndComp
 $Comp
-L taobao-c:C106,0603 C?
+L taobao-c:C106,0603 C2
 U 1 1 5D003198
 P 5100 2350
-F 0 "C?" H 5200 2400 50  0000 L CNN
+F 0 "C2" H 5200 2400 50  0000 L CNN
 F 1 "C106,0603" H 5200 2350 50  0000 L CNN
 F 2 "Capacitor_SMD:C_0603_1608Metric_Pad1.05x0.95mm_HandSolder" H 5100 2350 50  0001 C CNN
@@
 	4300 2450 4300 2550
 $Comp
-L power:GND #PWR?
+L power:GND #PWR0113
 U 1 1 5D22DD1F
 P 4300 2550
-F 0 "#PWR?" H 4300 2300 50  0001 C CNN
+F 0 "#PWR0113" H 4300 2300 50  0001 C CNN
 F 1 "GND" H 4400 2550 50  0000 L CNN
 F 2 "" H 4300 2550 50  0001 C CNN
@@
 $EndComp
 $Comp
-L taobao-c:C106,0603 C?
+L taobao-c:C106,0603 C1
 U 1 1 5D22DD29
 P 4300 2350
-F 0 "C?" H 4400 2400 50  0000 L CNN
+F 0 "C1" H 4400 2400 50  0000 L CNN
 F 1 "C106,0603" H 4400 2350 50  0000 L CNN
 F 2 "Capacitor_SMD:C_0603_1608Metric_Pad1.05x0.95mm_HandSolder" H 4300 2350 50  0001 C CNN
