File: hardware/MCP73831.kicad_pcb (KiCad board)
At the start: 2 copper layers, 11 parts, among them J1 PWR_SRC, J2 5V_OUT, J3 BAT, U1 MCP73831

Commit message: update,
Parts:
- added C1: C106,0603, Capacitor_SMD:C_0603_1608Metric_Pad1.05x0.95mm_HandSolder, F.Cu at (37.0, 26.2)
- renumbered C1 to C2
Connections:
- net VCC renamed VBUS
- C2 pad 1: Vbat -> +5V
Changed lines of the file:
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@@
     (tracks 56)
     (zones 0)
-    (modules 11)
+    (modules 12)
     (nets 10)
   )
@@
   (net 7 "Net-(R1-Pad1)")
   (net 8 "Net-(R2-Pad2)")
-  (net 9 VCC)
+  (net 9 VBUS)
   (net_class Default "This is the default net class."
     (clearance 0.2)
@@
     (add_net "Net-(R1-Pad1)")
     (add_net "Net-(R2-Pad2)")
-    (add_net VCC)
+    (add_net VBUS)
     (add_net Vbat)
+  )
+  (module Capacitor_SMD:C_0603_1608Metric_Pad1.05x0.95mm_HandSolder (layer F.Cu)
+    (at 37 26.2)
+    (descr "Capacitor SMD 0603 (1608 Metric), square (rectangular) end terminal, IPC_7351 nominal with elongated pad for handsoldering. (Body size source: http://www.tortai-tech.com/upload/download/2011102023233369053.pdf), generated with kicad-footprint-generator")
+    (tags "capacitor handsolder")
+    (attr smd)
+    (fp_text reference C1 (at 0 -1.43) (layer F.SilkS)
+      (effects (font (size 1 1) (thickness 0.15)))
+    )
+    (fp_text value C106,0603 (at 0 1.43) (layer F.Fab)
+      (effects (font (size 1 1) (thickness 0.15)))
+    )
+    (fp_text user %R (at 0 0) (layer F.Fab)
+      (effects (font (size 0.4 0.4) (thickness 0.06)))
+    )
+    (fp_line (start 1.65 0.73) (end -1.65 0.73) (layer F.CrtYd) (width 0.05))
+    (fp_line (start 1.65 -0.73) (end 1.65 0.73) (layer F.CrtYd) (width 0.05))
+    (fp_line (start -1.65 -0.73) (end 1.65 -0.73) (layer F.CrtYd) (width 0.05))
+    (fp_line (start -1.65 0.73) (end -1.65 -0.73) (layer F.CrtYd) (width 0.05))
+    (fp_line (start -0.171267 0.51) (end 0.171267 0.51) (layer F.SilkS) (width 0.12))
+    (fp_line (start -0.171267 -0.51) (end 0.171267 -0.51) (layer F.SilkS) (width 0.12))
+    (fp_line (start 0.8 0.4) (end -0.8 0.4) (layer F.Fab) (width 0.1))
+    (fp_line (start 0.8 -0.4) (end 0.8 0.4) (layer F.Fab) (width 0.1))
+    (fp_line (start -0.8 -0.4) (end 0.8 -0.4) (layer F.Fab) (width 0.1))
+    (fp_line (start -0.8 0.4) (end -0.8 -0.4) (layer F.Fab) (width 0.1))
+    (pad 2 smd roundrect (at 0.875 0) (size 1.05 0.95) (layers F.Cu F.Paste F.Mask) (roundrect_rratio 0.25)
+      (net 1 GND))
+    (pad 1 smd roundrect (at -0.875 0) (size 1.05 0.95) (layers F.Cu F.Paste F.Mask) (roundrect_rratio 0.25)
+      (net 2 Vbat))
+    (model ${KISYS3DMOD}/Capacitor_SMD.3dshapes/C_0603_1608Metric.wrl
+      (at (xyz 0 0 0))
+      (scale (xyz 1 1 1))
+      (rotate (xyz 0 0 0))
+    )
   )
   (module Connector_PinHeader_2.54mm:PinHeader_1x02_P2.54mm_Vertical (layer F.Cu)
@@
     (fp_line (start -0.635 -1.27) (end 1.27 -1.27) (layer F.Fab) (width 0.1))
     (pad 2 thru_hole oval (at 0 2.54 270) (size 1.7 1.7) (drill 1) (layers *.Cu *.Mask)
-      (net 9 VCC))
+      (net 9 VBUS))
     (pad 1 thru_hole rect (at 0 0 270) (size 1.7 1.7) (drill 1) (layers *.Cu *.Mask)
       (net 1 GND))
@@
       ))
     (pad 1 smd custom (at -0.65 0 270) (size 1 0.5) (layers F.Cu F.Mask)
-      (net 9 VCC) (zone_connect 2)
+      (net 9 VBUS) (zone_connect 2)
       (options (clearance outline) (anchor rect))
       (primitives
@@
     (tags "capacitor handsolder")
     (attr smd)
-    (fp_text reference C1 (at 0 -1.43) (layer F.SilkS)
+    (fp_text reference C2 (at 0 -1.43) (layer F.SilkS)
       (effects (font (size 1 1) (thickness 0.15)))
     )
@@
       (net 1 GND))
     (pad 1 smd roundrect (at -0.875 0) (size 1.05 0.95) (layers F.Cu F.Paste F.Mask) (roundrect_rratio 0.25)
-      (net 2 Vbat))
+      (net 3 +5V))
     (model ${KISYS3DMOD}/Capacitor_SMD.3dshapes/C_0603_1608Metric.wrl
       (at (xyz 0 0 0))

Commit message: update,
Routing:
- net +5V: track 5.93 -> 17.5 mm, vias 0 -> 1
- net GND: track 36.8 -> 40.4 mm
- net Vbat: track 12.1 -> 12.7 mm
